File: foc_controller/foc_controller.kicad_pcb (KiCad board)
At the start: 2 copper layers, 46 parts, among them J1 Conn_01x02, J1-Programmer1 Conn_01x05, J2 Conn_01x04, J3 Conn_01x03, J5 USB_C_Receptacle_USB2.0_16P, J6 Conn_01x02, U1 AZ1117-3.3, U2 INA4180A2IPWR, U4 AS5048B, U5 STM32G431KBUx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

Commit message: Circular rendition started.
Parts:
- removed D1, D2: PWR_LED, LED_SMD:LED_0603_1608Metric
- removed J1, J6: Conn_01x02, Connector_PinHeader_2.00mm:PinHeader_1x02_P2.00mm_Vertical
- removed J2: Conn_01x04, Connector_PinHeader_2.00mm:PinHeader_1x04_P2.00mm_Vertical
- removed J5: USB_C_Receptacle_USB2.0_16P, usb_connector_footprints:12402012E212A_AMP
- removed R1, R2: 1k5, Resistor_SMD:R_0603_1608Metric
- removed R4, R5: 5.1k, Resistor_SMD:R_0603_1608Metric
- removed SW1: ~, button_footprint:SMT_FS
- added ATA1: ~, Package_DFN_QFN:DFN-8-1EP_3x3mm_P0.5mm_EP1.65x2.38mm, F.Cu at (130.1, 48.2)
- added C22: 100nF, Capacitor_SMD:C_0603_1608Metric, F.Cu at (117.8, 38.8)
- added C23: 100nF, Capacitor_SMD:C_0603_1608Metric, F.Cu at (124.8, 39.0)
- added C24: 10u, Capacitor_SMD:C_0603_1608Metric, F.Cu at (109.0, 34.0)
- added C25: 22u, Capacitor_SMD:C_0603_1608Metric, F.Cu at (117.8, 37.2)
- added J4: Conn_01x04, Connector_PinHeader_2.00mm:PinHeader_1x04_P2.00mm_Vertical, F.Cu at (134.0, 42.0)
- added U6: AZ1117-5.0, custom:SOT-223_DIO, F.Cu at (114.0, 34.5)
- J1-Programmer1: footprint Connector_PinHeader_2.00mm:PinHeader_1x05_P2.00mm_Vertical -> Connector_PinHeader_1.27mm:PinHeader_1x05_P1.27mm_Vertical
- moved C16 68.0 mm to (127.8, 42.0)
- moved J1-Programmer1 58.5 mm to (130.8, 45.3), turned to 180 degrees
- moved U5 55.2 mm to (123.0, 52.7), turned to 45 degrees
- moved Y1 55.0 mm to (115.0, 57.0)
- moved C10 54.3 mm to (115.0, 59.5)
- moved Rshunt2 52.7 mm to (113.0, 41.5), turned to 180 degrees
- moved C9 52.6 mm to (111.8, 58.0), turned to 180 degrees
- moved C17 50.5 mm to (127.8, 39.0), turned to 0 degrees
- moved C18 49.4 mm to (124.8, 37.5), turned to 180 degrees
- moved C6 48.2 mm to (112.0, 53.0), turned to 0 degrees
- moved C14 48.2 mm to (127.8, 40.5)
- moved C15 48.2 mm to (127.8, 37.5)
- moved U2 46.4 mm to (108.5, 42.0), turned to 90 degrees
- moved Rshunt1 45.7 mm to (107.7, 47.0), turned to 0 degrees
- moved C3 44.9 mm to (106.5, 54.5), turned to -90 degrees
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Connections:
- net VBUS renamed +5V
- U5 pad 20: unconnected-(U5-PA10-Pad20) -> ATA6561_STBY
Routing:
- net +12V: track 11.6 -> 58.0 mm, vias 0 -> 3
- net UART2_TX: track 33.8 -> 0.00 mm, vias 2 -> 0
- net +5V: track 5.49 -> 38.9 mm, vias 0 -> 2
- net +3.3V: track 101.4 -> 68.9 mm
- net U_ADC1_IN15: track 29.3 -> 0.00 mm, vias 2 -> 0
- net V_ADC1_IN10: track 27.9 -> 0.00 mm, vias 2 -> 0
- net Net-(J1-Programmer1-Pin_2): track 24.9 -> 0.00 mm, vias 1 -> 0
- net UART2_RX: track 24.7 -> 0.00 mm, vias 2 -> 0
- net GND: track 92.5 -> 68.7 mm, vias 18 -> 9
- net USB_DM: track 23.2 -> 0.00 mm
- net USB_DP: track 22.5 -> 0.00 mm
- net NRST: track 24.9 -> 2.50 mm
- net I2C_SDA: track 19.5 -> 0.00 mm, vias 2 -> 0
- net W_ADC2_IN4: track 18.1 -> 0.00 mm, vias 2 -> 0
- net MOTOR_DIAG: track 17.9 -> 0.00 mm, vias 2 -> 0
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Other:
- board outline added: 34.5 x 32 mm

Commit message: More routing
Routing:
- net GND: track 68.7 -> 80.5 mm, vias 9 -> 13
- net OSC_IN: track 0.00 -> 10.1 mm
- net OSC_OUT: track 0.00 -> 8.49 mm
- net Net-(U3-VCP): track 0.00 -> 6.41 mm, vias 0 -> 2
- net +5V: track 38.9 -> 44.6 mm
- net CANH: track 0.00 -> 3.33 mm
- net CANL: track 0.00 -> 2.71 mm
- net PA2_TIM15_CH1: track 0.00 -> 2.12 mm, vias 0 -> 1
- net Wphase: track 27.2 -> 29.3 mm
- net PA6_TIM16_CH1: track 0.00 -> 1.62 mm, vias 0 -> 1
- net PB5_TIM17_CH1: track 0.00 -> 1.06 mm, vias 0 -> 1
- net (no net): track 1.00 -> 0.00 mm
- net +12V: track 58.0 -> 58.5 mm

Commit message: More routing
Parts:
- moved Rshunt1 0.72 mm to (107.0, 46.8)
Routing:
- net W_ADC2_IN4: track 0.00 -> 48.2 mm, vias 0 -> 2
- net U_ADC1_IN15: track 0.00 -> 37.4 mm, vias 0 -> 2
- net +3.3V: track 68.9 -> 101.3 mm, vias 2 -> 8
- net MOTOR_DIAG: track 0.00 -> 21.5 mm, vias 0 -> 2
- net V_ADC1_IN10: track 0.00 -> 20.5 mm, vias 0 -> 2
- net MOTOR_STDBY: track 3.90 -> 19.1 mm, vias 0 -> 2
- net PB6_TIM16_CH1N: track 0.00 -> 15.1 mm
- net PB7_TIM17_CH1N: track 0.00 -> 12.8 mm
- net Wphase: track 29.3 -> 17.1 mm, vias 0 -> 1
- net PA2_TIM15_CH1: track 2.12 -> 13.7 mm, vias 1 -> 2
- net Uphase: track 2.48 -> 12.8 mm, vias 0 -> 2
- net PB5_TIM17_CH1: track 1.06 -> 9.92 mm, vias 1 -> 2
- net Uout: track 8.36 -> 14.8 mm
- net Vout: track 18.2 -> 21.6 mm
- net GND: track 80.5 -> 83.3 mm, vias 13 -> 12
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
Commit message: Finished routing
Connections:
- U3 pad 6: PA2_TIM15_CH1N -> PA1_TIM15_CH1N
- U5 pad 11: PA6_TIM15_CH1 -> PA6_TIM16_CH1
Routing:
- net GND: track 83.3 -> 121.9 mm, vias 12 -> 15
- net NRST: track 2.50 -> 29.1 mm, vias 0 -> 1
- net PA1_TIM15_CH1N: track 0.00 -> 19.6 mm, vias 0 -> 2
- net PA6_TIM16_CH1: track 0.00 -> 19.3 mm, vias 0 -> 2
- net +3.3VA: track 4.51 -> 20.9 mm, vias 1 -> 2
- net I2C_SDA: track 0.00 -> 13.4 mm, vias 0 -> 2
- net I2C_SCL: track 0.00 -> 12.8 mm, vias 0 -> 2
- net Wphase: track 17.1 -> 29.4 mm, vias 1 -> 2
- net ATA6561_STBY: track 0.00 -> 10.5 mm, vias 0 -> 2
- net Uout: track 14.8 -> 5.07 mm
- net Net-(J1-Programmer1-Pin_2): track 0.00 -> 9.74 mm, vias 0 -> 1
- net Net-(J1-Programmer1-Pin_1): track 0.00 -> 8.90 mm, vias 0 -> 1
- net UART2_TX: track 0.00 -> 8.55 mm
- net UART2_RX: track 0.00 -> 8.23 mm
- net MOTOR_STDBY: track 19.1 -> 26.7 mm
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Other:
- outline, holes or cut-outs redrawn
